Commit message: Codebase cleanup: removed files for real robot movement now we can simulate in gazebo, Rviz and use SLAM toolbox to map the environment Initial files for PPO reinforcement learning algorithm to train the robot to move in the environment.

File: urdf/martha.urdf (robot description, URDF)
Before this commit: robot Martha, 6 links, 5 joints
Joints:
- joint base_back_left_wheel_joint: type continuous -> fixed
- joint base_back_right_wheel_joint: type continuous -> fixed
- joint base_front_left_wheel_joint: type continuous -> fixed
- joint base_front_right_wheel_joint: type continuous -> fixed
