File: pcb/martha_circuits/_restore_backup_2026-07-23T15-24-39-500/martha_circuits.kicad_pcb (KiCad board)
At the start: 2 copper layers, 140 x 200 mm, 16 parts, among them J1 Conn_01x06, J2 Conn_01x06, J3 Conn_01x06, J4 Conn_01x06, J5 IMU, J6 Conn_01x02_Dean, SW1 SW_SPST, U5 LM339

Commit message: Schematics and PCB development
Connections:
- R1 pad 2: Net-(U0-D23) -> Net-(U0-D4)
- U0 pad 10: Net-(J1-Pin_6) -> Net-(U0-D27)
- U0 pad 11: Net-(J1-Pin_5) -> Net-(U0-D14)
- U0 pad 12: Net-(J3-Pin_6) -> unconnected-(U0-D12-Pad12)
- U0 pad 13: Net-(J3-Pin_5) -> Net-(U0-D13)
- U0 pad 2: Net-(J2-Pin_6) -> Net-(J2-Pin_5)
- U0 pad 23: Net-(U0-D5) -> unconnected-(U0-D5-Pad23)
- U0 pad 26: Net-(J5-Pin_3) -> Net-(J5-Pin_4)
- U0 pad 29: Net-(J5-Pin_4) -> Net-(J5-Pin_3)
- U0 pad 3: Net-(J2-Pin_5) -> Net-(J2-Pin_6)
- U0 pad 4: unconnected-(U0-D34-Pad4) -> Net-(J1-Pin_5)
- U0 pad 5: unconnected-(U0-D35-Pad5) -> Net-(J1-Pin_6)
- U0 pad 6: Net-(U0-D32) -> Net-(J3-Pin_5)
- U0 pad 7: Net-(U0-D33) -> Net-(J3-Pin_6)
- U1 pad 4: Net-(U0-D26) -> Net-(U0-D25)
- U1 pad 5: Net-(U0-D25) -> Net-(U0-D26)
- U2 pad 4: Net-(U0-D33) -> Net-(U0-D27)
- U2 pad 5: Net-(U0-D32) -> Net-(U0-D14)
- U3 pad 4: Net-(U0-D4) -> Net-(U0-RX2(16))
- U3 pad 5: Net-(U0-RX2(16)) -> Net-(U0-TX2(17))
- U4 pad 4: Net-(U0-TX2(17)) -> Net-(U0-D23)
- U4 pad 5: Net-(U0-D5) -> Net-(U0-D13)
- U5 pad 1: Net-(U0-D23) -> Net-(U0-D4)
- U5 pad 13: Net-(U0-D23) -> Net-(U0-D4)
- U5 pad 14: Net-(U0-D23) -> Net-(U0-D4)
- U5 pad 2: Net-(U0-D23) -> Net-(U0-D4)
Routing:
- net Net-(U0-D13): track 0.00 -> 103.1 mm
- net Net-(U0-D33): track 102.7 -> 0.00 mm
- net Net-(U0-D5): track 101.5 -> 0.00 mm
- net Net-(U0-D32): track 99.6 -> 0.00 mm
- net Net-(U0-D27): track 0.00 -> 87.2 mm
- net Net-(U0-D14): track 0.00 -> 84.6 mm
- net Net-(U0-TX2(17)): track 99.9 -> 47.0 mm
- net Net-(U0-D4): track 46.7 -> 84.4 mm
- net Net-(U0-D23): track 86.5 -> 102.7 mm
- net Net-(J2-Pin_5): track 136.8 -> 123.2 mm
- net Net-(J2-Pin_6): track 135.4 -> 125.5 mm
- net Net-(U0-RX2(16)): track 51.0 -> 45.1 mm
- net Net-(U0-D26): track 64.8 -> 58.9 mm
- net Net-(J1-Pin_6): track 89.3 -> 92.6 mm
- net Net-(J3-Pin_6): track 121.4 -> 118.1 mm
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