File: pcb/martha_circuits/_restore_backup_2026-07-23T15-24-39-500/martha_circuits.kicad_sch (KiCad schematic)
At the start: 17 parts, among them J1 Conn_01x06, J2 Conn_01x06, J3 Conn_01x06, J4 Conn_01x06, J5 IMU, J6 Conn_01x02_Dean, SW1 SW_SPST, U5 LM339

Commit message: Schematics and PCB development
Parts:
- removed R2, R3: R, Resistor_THT:R_Axial_DIN0207_L6.3mm_D2.5mm_P7.62mm_Horizontal, symbol Device:R
- R1: value 100k -> R
Connections:
- net at J1.5 (Pin_5): now also U0.5 (D35); no longer U0.11 (D14)
- net at J1.6 (Pin_6): now also U0.4 (D34); no longer U0.10 (D27)
- net at U1.4 (IN1): now also U0.8 (D25); no longer U0.9 (D26)
- net at U1.5 (IN2): now also U0.9 (D26); no longer U0.8 (D25)
