File: pcb/martha_circuits/martha_circuits.kicad_pcb (KiCad board)
At the start: 2 copper layers, 140 x 200 mm, 16 parts, among them J1 Conn_01x06, J2 Conn_01x06, J3 Conn_01x06, J4 Conn_01x06, J5 IMU, J6 Conn_01x02_Dean, SW1 SW_SPST, U5 LM339

Commit message: Some corrections from Miti
Parts:
- added C1: 10nf, Capacitor_THT:C_Disc_D5.0mm_W2.5mm_P2.50mm, F.Cu at (251.0, 89.7)
- added C2: 10nf, Capacitor_THT:C_Disc_D5.0mm_W2.5mm_P2.50mm, F.Cu at (251.0, 93.8)
- added D1: LED, LED_THT:LED_D5.0mm, F.Cu at (244.0, 85.5)
- added D2: LED, LED_THT:LED_D5.0mm, F.Cu at (244.0, 93.0)
- added D3: LED, LED_THT:LED_D5.0mm, F.Cu at (244.0, 100.4)
- added D4: LED, LED_THT:LED_D5.0mm, F.Cu at (244.0, 107.9)
- added Q1: IRF4905, Package_TO_SOT_THT:TO-220-3_Vertical, F.Cu at (252.2, 85.7)
- added R1: 47k, Resistor_THT:R_Axial_DIN0207_L6.3mm_D2.5mm_P7.62mm_Horizontal, F.Cu at (232.3, 83.8)
- added R10: R, Resistor_THT:R_Axial_DIN0207_L6.3mm_D2.5mm_P7.62mm_Horizontal, F.Cu at (232.3, 116.2)
- added R2: R, Resistor_THT:R_Axial_DIN0207_L6.3mm_D2.5mm_P7.62mm_Horizontal, F.Cu at (232.3, 87.8)
- added R3: R, Resistor_THT:R_Axial_DIN0207_L6.3mm_D2.5mm_P7.62mm_Horizontal, F.Cu at (232.3, 91.9)
- added R5: 39k, Resistor_THT:R_Axial_DIN0207_L6.3mm_D2.5mm_P7.62mm_Horizontal, F.Cu at (232.3, 95.9)
- added R6: 10k, Resistor_THT:R_Axial_DIN0207_L6.3mm_D2.5mm_P7.62mm_Horizontal, F.Cu at (232.3, 100.0)
- added R7: R, Resistor_THT:R_Axial_DIN0207_L6.3mm_D2.5mm_P7.62mm_Horizontal, F.Cu at (232.3, 104.0)
- added R8: R, Resistor_THT:R_Axial_DIN0207_L6.3mm_D2.5mm_P7.62mm_Horizontal, F.Cu at (232.3, 108.1)
- added R9: R, Resistor_THT:R_Axial_DIN0207_L6.3mm_D2.5mm_P7.62mm_Horizontal, F.Cu at (232.3, 112.1)
- R4: renamed from R1; value R -> 100k
- renumbered J6 to J1, J3 to J2, J1 to J3, J5 to J4, J4 to J5, J2 to J6, U3 to U1, U1 to U2, U5 to U3, U0 to U4, U2 to U5, U4 to U6
Connections:
- J1 pad 1: Net-(J6-Pin_1) (its old number) -> Net-(J1-Pin_1)
- SW1 pad 1: Net-(J6-Pin_1) (its old number) -> Net-(Q1-S)
- U1 pad 8: unconnected-(U3-FAULT-Pad8) -> FAULT3
- U2 pad 8: unconnected-(U1-FAULT-Pad8) -> FAULT1
- U5 pad 8: unconnected-(U2-FAULT-Pad8) -> FAULT2
- U6 pad 8: unconnected-(U4-FAULT-Pad8) -> FAULT4
Routing:
- net Net-(J6-Pin_1) (its old number): track 14.1 -> 0.00 mm
- net Net-(J1-Pin_1): track 0.00 -> 14.1 mm

Commit message: - First PPO implementation (Read the Code) - PCB finished (Must ask teacher for corrections)
Parts:
- removed U6: ~, Pololu_Driver:MPQ6612A
- added HEX M4: MountingHole_4.3mm_M4, MountingHole:MountingHole_4.3mm_M4, F.Cu at (54.1, 170.3)
- added HEX M4: MountingHole_4.3mm_M4, MountingHole:MountingHole_4.3mm_M4, F.Cu at (155.1, 170.3)
- added HEX M4: MountingHole_4.3mm_M4, MountingHole:MountingHole_4.3mm_M4, F.Cu at (54.1, 55.4)
- added U0: ~, ESP32_dev_module:ESP32_DevKit_30Pin, F.Cu at (104.9, 111.2)
- HEX M4: renamed from REF**
- J1: value Conn_01x02_Dean -> Conn_01x06; footprint My_Components:DEANS -> My_Components:PinHeader_1x06_P2.54mm_Horizontal_Mirrored
- J2: footprint Connector_PinHeader_2.54mm:PinHeader_1x06_P2.54mm_Horizontal -> My_Components:PinHeader_1x06_P2.54mm_Horizontal_Mirrored; moved to F.Cu
- J3: footprint Connector_PinHeader_2.54mm:PinHeader_1x06_P2.54mm_Horizontal -> My_Components:PinHeader_1x06_P2.54mm_Horizontal_Mirrored
- J4: value IMU -> Conn_01x06; footprint Connector_PinHeader_2.54mm:PinHeader_1x08_P2.54mm_Vertical -> My_Components:PinHeader_1x06_P2.54mm_Horizontal_Mirrored
- J5: value Conn_01x06 -> Battery; footprint Connector_PinHeader_2.54mm:PinHeader_1x06_P2.54mm_Horizontal -> My_Components:DEANS; moved to F.Cu
- J6: value Conn_01x06 -> IMU; footprint Connector_PinHeader_2.54mm:PinHeader_1x06_P2.54mm_Horizontal -> Connector_PinHeader_2.54mm:PinHeader_1x08_P2.54mm_Vertical
- U1, U2: moved to F.Cu
- U3: value LM339 -> ~; footprint Package_DIP:DIP-14_W7.62mm -> Pololu_Driver:MPQ6612A
- U4: footprint ESP32_dev_module:ESP32_DevKit_30Pin -> Pololu_Driver:MPQ6612A
- U5: value ~ -> LM339; footprint Pololu_Driver:MPQ6612A -> Package_DIP:DIP-14_W7.62mm; moved to F.Cu
- moved HEX M4 218.3 mm to (155.1, 55.4)
- moved J2 194.1 mm to (145.3, 51.1)
- moved Q1 188.9 mm to (64.3, 104.3)
- moved D1 182.5 mm to (61.5, 83.1), turned to 90 degrees
- moved R7 173.1 mm to (61.5, 75.8), turned to 90 degrees
- moved R1 172.2 mm to (64.3, 121.6), turned to 90 degrees
- moved D3 158.7 mm to (90.7, 141.5), turned to -90 degrees
- moved R9 146.5 mm to (90.7, 149.4), turned to -90 degrees
- moved J5 140.7 mm to (53.0, 113.0), turned to 0 degrees
- moved J3 134.5 mm to (67.8, 174.2)
- moved D2 121.6 mm to (123.1, 79.5), turned to 90 degrees
- moved U1 117.6 mm to (80.5, 74.5), turned to -90 degrees
- moved SW1 116.5 mm to (53.0, 104.3), turned to 0 degrees
- moved R8 115.0 mm to (123.1, 72.2), turned to 90 degrees
- moved C2 111.7 mm to (139.6, 101.7), turned to 90 degrees
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Connections:
- net Net-(C2-Pad1) renamed Batt_Charge
- C1 pad 1: +5V2 -> +5V4
- J1 pad 2: GND -> Net-(J1-Pin_2)
- J2 pad 4: +5V3 -> +5V2
- J3 pad 4: +5V1 -> +5V3
- J4 pad 1: +3.3V -> Net-(J4-Pin_1)
- J4 pad 2: GND -> Net-(J4-Pin_2)
- J4 pad 3: Net-(J4-Pin_3) -> GND
- J4 pad 4: Net-(J4-Pin_4) -> +5V4
- J4 pad 5: (no net) -> Net-(J4-Pin_5)
- J4 pad 6: (no net) -> Net-(J4-Pin_6)
- J5 pad 2: Net-(J5-Pin_2) -> GND
- J6 pad 1: Net-(J6-Pin_1) -> +3.3V
- J6 pad 2: Net-(J6-Pin_2) -> GND
- J6 pad 3: GND -> Net-(J6-Pin_3)
- J6 pad 4: +5V2 -> Net-(J6-Pin_4)
- J6 pad 5: Net-(J6-Pin_5) -> (no net)
- J6 pad 6: Net-(J6-Pin_6) -> (no net)
- Q1 pad 2: Net-(J1-Pin_1) -> Net-(Q1-D)
- Q1 pad 3: Net-(Q1-S) -> +12V
- R10 pad 2: +5V3 -> +5V4
- R2 pad 1: +5V2 -> +5V4
- R4 pad 1: +3.3V -> +5V4
- R4 pad 2: Net-(U4-D23) -> Net-(U0-D23)
- RV1 pad 1: +5V2 -> +5V4
- SW1 pad 1: Net-(Q1-S) -> Net-(J5-Pin_1)
- SW1 pad 2: +12V -> Net-(Q1-D)
- U1 pad 12: Net-(J2-Pin_2) -> Net-(J1-Pin_2)
- U1 pad 13: Net-(J2-Pin_1) -> Net-(J1-Pin_1)
- U1 pad 3: +5V3 -> +5V1
- U1 pad 4: Net-(U1-IN1) -> Net-(U0-D27)
- U1 pad 5: Net-(U1-IN2) -> Net-(U0-D14)
- U1 pad 6: Net-(U1-SLEEP) -> Net-(U0-TX2(17))
- U1 pad 8: FAULT3 -> FAULT1
- U2 pad 12: Net-(J3-Pin_2) -> Net-(J2-Pin_2)
- U2 pad 13: Net-(J3-Pin_1) -> Net-(J2-Pin_1)
- U2 pad 3: +5V1 -> +5V2
- U2 pad 4: Net-(U2-IN1) -> Net-(U0-D32)
- U2 pad 5: Net-(U2-IN2) -> Net-(U0-D33)
- U2 pad 6: Net-(U1-SLEEP) -> Net-(U0-TX2(17))
- U2 pad 8: FAULT1 -> FAULT2
- U3 pad 1: Net-(U4-D23) -> unconnected-(U3-VM-Pad1)
- U3 pad 10: Net-(U3C--) -> unconnected-(U3-ISET-Pad10)
- U3 pad 11: VD -> +12V
- U3 pad 12: GND -> Net-(J3-Pin_2)
- U3 pad 13: Net-(U4-D23) -> Net-(J3-Pin_1)
- U3 pad 14: Net-(U4-D23) -> GND
- U3 pad 2: Net-(U4-D23) -> GND
- U3 pad 3: +5V2 -> +5V3
- U3 pad 4: Net-(U3A--) -> Net-(U0-D15)
- U3 pad 5: VD -> Net-(U0-D2)
- U3 pad 6: Net-(U2-ViSEN) -> Net-(U0-TX2(17))
- U3 pad 7: VD -> Net-(U3-ViSEN)
- U3 pad 8: Net-(U1-ViSEN) -> FAULT3
- U3 pad 9: VD -> unconnected-(U3-OC_ADJ-Pad9)
- U4 pad 10: Net-(J3-Pin_6) -> unconnected-(U4-ISET-Pad10)
- U4 pad 11: Net-(J3-Pin_5) -> +12V
- U4 pad 12: Net-(J2-Pin_6) -> Net-(J4-Pin_2)
- U4 pad 13: Net-(J2-Pin_5) -> Net-(J4-Pin_1)
- U4 pad 2: Net-(J6-Pin_6) -> GND
- U4 pad 3: Net-(J6-Pin_5) -> +5V4
- U4 pad 4: unconnected-(U4-D34-Pad4) -> Net-(U0-D18)
- U4 pad 5: unconnected-(U4-D35-Pad5) -> Net-(U0-D19)
- U4 pad 6: Net-(U4-D32) -> Net-(U0-TX2(17))
- U4 pad 7: Net-(U4-D33) -> Net-(U4-ViSEN)
- U4 pad 8: Net-(U2-IN2) -> FAULT4
- U4 pad 9: Net-(U2-IN1) -> unconnected-(U4-OC_ADJ-Pad9)
- U5 pad 1: unconnected-(U5-VM-Pad1) -> Net-(U0-D23)
- U5 pad 10: unconnected-(U5-ISET-Pad10) -> Net-(U3-ViSEN)
- U5 pad 11: +12V -> VD
- U5 pad 12: Net-(J6-Pin_2) -> GND
- U5 pad 13: Net-(J6-Pin_1) -> Net-(U0-D23)
- U5 pad 14: GND -> Net-(U0-D23)
- U5 pad 2: GND -> Net-(U0-D23)
- U5 pad 3: +5V2 -> +5V4
- U5 pad 4: Net-(U4-D33) -> Net-(U1-ViSEN)
- U5 pad 5: Net-(U4-D32) -> VD
- U5 pad 6: Net-(U1-SLEEP) -> Net-(U2-ViSEN)
- U5 pad 7: Net-(U3A--) -> VD
- U5 pad 8: FAULT2 -> Net-(U4-ViSEN)
- U5 pad 9: unconnected-(U5-OC_ADJ-Pad9) -> VD
Routing:
- net +12V: track 433.2 -> 48.1 mm
- net Net-(U1-SLEEP): track 316.3 -> 0.00 mm
- net Net-(U0-TX2(17)): track 0.00 -> 210.1 mm
- net Net-(J5-Pin_5): track 140.8 -> 0.00 mm
- net Net-(J5-Pin_6): track 138.5 -> 0.00 mm
- net Net-(J6-Pin_5): track 136.8 -> 0.00 mm
- net Net-(J6-Pin_6): track 135.4 -> 0.00 mm
- net Net-(U4-D33): track 102.7 -> 0.00 mm
- net Net-(U4-D5): track 101.5 -> 0.00 mm
- net Net-(U4-TX2(17)): track 99.9 -> 0.00 mm
- net Net-(U4-D32): track 99.6 -> 0.00 mm
- net Net-(U3-ViSEN): track 0.00 -> 87.2 mm
- net Net-(U4-D23): track 86.5 -> 0.00 mm
- net Net-(J1-Pin_5): track 0.00 -> 82.3 mm
- net Net-(J4-Pin_5): track 0.00 -> 81.6 mm
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- added copper zone on F.Cu, net +12V
- added copper zone on F.Cu, net GND
- added copper zone on F.Cu, net Net-(Q1-D)
Other:
- board size 140 x 200 mm -> 115 x 129 mm
