File: pcb/martha_circuits/martha_circuits.kicad_sch (KiCad schematic)
At the start: 17 parts, among them J1 Conn_01x06, J2 Conn_01x06, J3 Conn_01x06, J4 Conn_01x06, J5 IMU, J6 Conn_01x02_Dean, SW1 SW_SPST, U5 LM339

Commit message: Some corrections from Miti
Parts:
- added C1, C2: 10nf, Capacitor_THT:C_Disc_D5.0mm_W2.5mm_P2.50mm, symbol Device:C
- added D1, D2, D3, D4: LED, LED_THT:LED_D5.0mm, symbol Device:LED
- added Q1: IRF4905, Package_TO_SOT_THT:TO-220-3_Vertical, symbol Transistor_FET:IRF4905
- added R1: 47k, Resistor_THT:R_Axial_DIN0207_L6.3mm_D2.5mm_P7.62mm_Horizontal, symbol Device:R
- added R10, R7, R8, R9: R, Resistor_THT:R_Axial_DIN0207_L6.3mm_D2.5mm_P7.62mm_Horizontal, symbol Device:R
- added R5: 39k, Resistor_THT:R_Axial_DIN0207_L6.3mm_D2.5mm_P7.62mm_Horizontal, symbol Device:R
- added R6: 10k, Resistor_THT:R_Axial_DIN0207_L6.3mm_D2.5mm_P7.62mm_Horizontal, symbol Device:R
- renumbered J6 to J1, J3 to J2, J1 to J3, J5 to J4, J4 to J5, J2 to J6, R1 to R4, U3 to U1, U1 to U2, U5 to U3, U0 to U4, U2 to U5, U4 to U6
Connections:
- net +12V: now also R5.1
- net +5V1: now also R7.2
- net +5V2: now also C1.1, R8.2
- net +5V3: now also R10.2, R9.2
- net GND: now also C1.2, C2.2, R1.1, R6.2
- net at J1.1 (Pin_1): now also Q1.2 (D); no longer SW1.1 (A)
- net FAULT3: now reaches U1.8 (FAULT)
- net FAULT3: now also D3.1 (K)
- net FAULT1: now reaches U2.8 (FAULT)
- net FAULT1: now also D1.1 (K)
- net FAULT4: now reaches U6.8 (FAULT)
- net FAULT4: now also D4.1 (K)
- net FAULT2: now reaches U5.8 (FAULT)
- net FAULT2: now also D2.1 (K)
- new net: Q1.1 (G), R1.2
- new net: Q1.3 (S), SW1.1 (A)
- new net: D2.2 (A), R8.1
- new net: D1.2 (A), R7.1
- new net: D4.2 (A), R10.1
- new net: C2.1, R5.2, R6.1
- new net: D3.2 (A), R9.1
Other:
- moved on the sheet: R2, R3, RV1, SW1, U3E

Commit message: - First PPO implementation (Read the Code) - PCB finished (Must ask teacher for corrections)
Parts:
- J1: renamed from J3; footprint Connector_PinHeader_2.54mm:PinHeader_1x06_P2.54mm_Horizontal -> My_Components:PinHeader_1x06_P2.54mm_Horizontal_Mirrored
- J2: renamed from J6; footprint Connector_PinHeader_2.54mm:PinHeader_1x06_P2.54mm_Horizontal -> My_Components:PinHeader_1x06_P2.54mm_Horizontal_Mirrored
- J3: renamed from J2; footprint Connector_PinHeader_2.54mm:PinHeader_1x06_P2.54mm_Horizontal -> My_Components:PinHeader_1x06_P2.54mm_Horizontal_Mirrored
- J4: renamed from J5; footprint Connector_PinHeader_2.54mm:PinHeader_1x06_P2.54mm_Horizontal -> My_Components:PinHeader_1x06_P2.54mm_Horizontal_Mirrored
- renumbered J1 to J5, J4 to J6, U4 to U0, U2 to U1, U5 to U2, U1 to U3, U6 to U4, U3 to U5
Connections:
- net +12V: now also Q1.3 (S); no longer SW1.2 (B)
- net +3.3V: no longer R4.1
- net +5V2: no longer C1.1, R2.1, RV1.1, U5.3 (V+)
- net +5V3: no longer R10.2
- net +5V4: now also C1.1, R10.2, R2.1, R4.1, RV1.1, U5.3 (V+)
- net at J4.5 (Pin_5): now also U0.26 (D21); no longer U0.24 (D18)
- net at J4.6 (Pin_6): now also U0.29 (D22); no longer U0.25 (D19)
- net at J2.5 (Pin_5): now also U0.2 (VP(36)); no longer U0.3 (VN(39))
- net at J2.6 (Pin_6): now also U0.3 (VN(39)); no longer U0.2 (VP(36))
- net at J1.5 (Pin_5): now also U0.12 (D12); no longer U0.11 (D14)
- net at J1.6 (Pin_6): now also U0.13 (D13); no longer U0.10 (D27)
- net at J3.5 (Pin_5): now also U0.20 (D4); no longer U0.13 (D13)
- net at J3.6 (Pin_6): now also U0.21 (RX2(16)); no longer U0.12 (D12)
- net at Q1.2 (D): now also SW1.2 (B); no longer J5.1 (Pin_1)
- net at SW1.1 (A): now also J5.1 (Pin_1); no longer Q1.3 (S)
- net Batt_Charge: now reaches C2.1, R5.2, R6.1
- net Batt_Charge: now also U0.4 (D34)
- net at J6.3 (Pin_3): now also U0.9 (D26); no longer U0.26 (D21)
- net at J6.4 (Pin_4): now also U0.8 (D25); no longer U0.29 (D22)
- net at U3.4 (IN1): now also U0.18 (D15); no longer U0.20 (D4)
- net at U3.5 (IN2): now also U0.19 (D2); no longer U0.21 (RX2(16))
- net at U1.6 (SLEEP), U2.6 (SLEEP), U3.6 (SLEEP)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: now also U0.22 (TX2(17)); no longer U0.19 (D2)
- net at U3.7 (ViSEN): now also U5.10 (-); no longer U5.8 (-)
- net at U1.4 (IN1): now also U0.10 (D27); no longer U0.9 (D26)
- net at U1.5 (IN2): now also U0.11 (D14); no longer U0.8 (D25)
- net at U1.7 (ViSEN): now also U5.4 (-); no longer U5.6 (-)
- net at U2.7 (ViSEN): now also U5.6 (-); no longer U5.4 (-)
- net at U4.4 (IN1): now also U0.24 (D18); no longer U0.22 (TX2(17))
- net at U4.5 (IN2): now also U0.25 (D19); no longer U0.23 (D5)
- net at U4.7 (ViSEN): now also U5.8 (-); no longer U5.10 (-)
- net at U2.4 (IN1): now also U0.6 (D32); no longer U0.7 (D33)
- net at U2.5 (IN2): now also U0.7 (D33); no longer U0.6 (D32)
Other:
- moved on the sheet: J5, Q1, R1, SW1, U5A, U5B, U5C, U5D
