File: pcb/martha_circuits/martha_circuits.kicad_sch (KiCad schematic)
At the start: 31 parts, among them J1 Conn_01x06, J2 Conn_01x06, J3 Conn_01x06, J4 Conn_01x06, J5 Conn_01x02_Dean, J6 IMU, Q1 IRF4905, SW1 SW_SPST, U5 LM339

Commit message: Learn obstacle avoidance: drop the OOB death, dense penalty, mastery curriculum
The policy plateaued on medium/long goals and out_of_bounds stayed high because
it was never actually learning to avoid obstacles. Three coupled causes, each
addressed here.

1. out_of_bounds was terminal at the 0.45 m inflated clearance, so the robot
   died the moment it entered the band, ~0.2 m before its 0.58x0.41 m footprint
   could touch anything. It never experienced getting close and recovering, so
   avoidance was learned only from sparse terminal deaths. out_of_bounds is no
   longer terminal: only a real bumper contact (or goal/timeout/stagnation) ends
   an episode. In the band the geodesic distance is undefined, so the last
   finite distance is frozen to keep shaping bounded; out_of_bounds is retained
   in the info dict purely as a near-obstacle diagnostic.

2. The clearance penalty was tiny and linear, negligible against the terminal.
   It is now the main obstacle signal: zero at 0.65 m and growing quadratically
   to laser_penalty_scale (0.10) at contact, so passing close is cheap
   (-0.005/step at 0.5 m) while nearly touching is strongly discouraged
   (-0.07/step at 0.1 m). Combined with removing the OOB death, the policy can
   now learn to thread close without touching.

3. The curriculum advanced on fixed episode fractions, outpacing avoidance, so
   the goals hardened before the policy was ready. CurriculumScheduler now
   raises the distance ceiling by mastery: it advances only when the rolling
   success over a full window clears curriculum_success_threshold (0.55), with a
   per-level episode cap as a stall fallback. curriculum_easy/medium/full_fraction
   are replaced by curriculum_success_threshold/window/min_episodes/max_episodes.

Test suite in the ros2_humble container: 178 passed. The 2 remaining failures
in test_shared_training predate this work.

Co-Authored-By: Claude Opus 4.8 <noreply@anthropic.com>
Parts:
- R10, R7, R8, R9: value R -> 1k
Connections:
- net +5V: no longer names the net of U0.15 (VIN)
Changed lines of the file:
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@@
 	(wire
 		(pts
+			(xy 78.74 146.05) (xy 191.77 146.05)
+		)
+		(stroke
+			(width 0)
+			(type default)
+		)
+	)
+	(wire
+		(pts
 			(xy 86.36 17.78) (xy 86.36 19.05)
 		)
@@
 	(wire
 		(pts
-			(xy 78.74 146.05) (xy 191.77 146.05)
-		)
-		(stroke
-			(width 0)
-			(type default)
-		)
-	)
-	(wire
-		(pts
 			(xy 128.27 72.39) (xy 128.27 83.82)
 		)
@@
 	(wire
 		(pts
-			(xy 128.27 114.3) (xy 130.81 114.3)
-		)
-		(stroke
-			(width 0)
-			(type default)
-		)
-	)
-	(wire
-		(pts
 			(xy 120.65 96.52) (xy 130.81 96.52)
 		)
@@
 			)
 		)
-		(property "Value" "R"
+		(property "Value" "1k"
 			(at 248.666 24.13 0)
 			(show_name no)
@@
 	)
 	(symbol
-		(lib_id "power:+5V")
-		(at 128.27 114.3 90)
-		(unit 1)
-		(body_style 1)
-		(exclude_from_sim no)
-		(in_bom yes)
-		(on_board yes)
-		(in_pos_files yes)
-		(dnp no)
-		(fields_autoplaced yes)
-		(property "Reference" "#PWR024"
-			(at 132.08 114.3 0)
-			(hide yes)
-			(show_name no)
-			(do_not_autoplace no)
-			(effects
-				(font
-					(size 1.27 1.27)
-				)
-			)
-		)
-		(property "Value" "+5V"
-			(at 124.46 114.2999 90)
-			(show_name no)
-			(do_not_autoplace no)
-			(effects
-				(font
-					(size 1.27 1.27)
-				)
-				(justify left)
-			)
-		)
-		(property "Footprint" ""
-			(at 128.27 114.3 0)
-			(hide yes)
-			(show_name no)
-			(do_not_autoplace no)
-			(effects
-				(font
-					(size 1.27 1.27)
-				)
-			)
-		)
-		(property "Datasheet" ""
-			(at 128.27 114.3 0)
-			(hide yes)
-			(show_name no)
-			(do_not_autoplace no)
-			(effects
-				(font
-					(size 1.27 1.27)
-				)
-			)
-		)
-		(property "Description" "Power symbol creates a global label with name \"+5V\""
-			(at 128.27 114.3 0)
-			(hide yes)
-			(show_name no)
-			(do_not_autoplace no)
-			(effects
-				(font
-					(size 1.27 1.27)
-				)
-			)
-		)
-		(pin "1"
-		)
-		(instances
-			(project "martha_circuits"
-				(path "/8a0047e5-3410-40b2-9332-77237a152757"
-					(reference "#PWR024")
-					(unit 1)
-				)
-			)
-		)
-	)
-	(symbol
 		(lib_id "power:+12V")
 		(at 50.8 59.69 0)
@@
 			)
 		)
-		(property "Value" "R"
+		(property "Value" "1k"
 			(at 237.236 24.13 0)
 			(show_name no)
@@
 			)
 		)
-		(property "Value" "R"
+		(property "Value" "1k"
 			(at 271.526 24.13 0)
 			(show_name no)
@@
 			)
 		)
-		(property "Value" "R"
+		(property "Value" "1k"
 			(at 260.096 24.13 0)
 			(show_name no)
